Commit message: bullet push world bug free

File: aml_robot/src/aml_robot/bullet/models/box_push_setup/plane.urdf (robot description, URDF)
Before this commit: robot plane.urdf, 1 links, 0 joints
Links:
- link planeLink: geometry collision box size=30 30 0.01; visual mesh filename=plane.obj scale=1 1 1
