Commit message: Added sawyer gripper controller

File: aml_sawyer_sim/sawyer_sim_description/urdf/sawyer.transmission.xacro (robot description, xacro)
@@ -82,4 +82,24 @@
       </actuator>
     </transmission>
+    <transmission name="r_gripper_l_finger_trans">
+      <type>transmission_interface/SimpleTransmission</type>
+      <joint name="r_gripper_l_finger_joint">
+        <hardwareInterface>EffortJointInterface</hardwareInterface>
+      </joint>
+      <actuator name="r_gripper_l_finger_motor">
+        <mechanicalReduction>1</mechanicalReduction>
+        <hardwareInterface>EffortJointInterface</hardwareInterface>
+      </actuator>
+    </transmission>
+    <transmission name="r_gripper_r_finger_trans">
+      <type>transmission_interface/SimpleTransmission</type>
+      <joint name="r_gripper_r_finger_joint">
+        <hardwareInterface>EffortJointInterface</hardwareInterface>
+      </joint>
+      <actuator name="r_gripper_r_finger_motor">
+        <mechanicalReduction>1</mechanicalReduction>
+        <hardwareInterface>EffortJointInterface</hardwareInterface>
+      </actuator>
+    </transmission>
   </xacro:macro>
 </robot>

File: aml_sawyer_sim/sawyer_sim_description/urdf/sawyer.urdf.xacro (robot description, xacro)
@@ -440,4 +440,25 @@
       <child link="screen"/>
     </joint>
+    <link name="head_display">
+      <visual>
+	<origin rpy="0 0 0" xyz="0 0 0.017"/>
+	<geometry>
+          <box size="0.24 0.14 0.001"/>
+	</geometry>
+	<material name="black">
+          <color rgba="0 0 0 1"/>
+	</material>
+      </visual>
+      <inertial>
+	<origin rpy="0 0 0" xyz="0 0 0"/>
+	<mass value="0.0001"/>
+	<inertia ixx="1e-08" ixy="0" ixz="0" iyy="1e-08" iyz="0" izz="1e-08"/>
+      </inertial>
+    </link>
+    <joint name="head_display_joint" type="fixed">
+      <origin rpy="0 0 0" xyz="0.0 0.0 -0.016"/>
+      <parent link="screen"/>
+      <child link="head_display"/>
+    </joint>
     <link name="head_camera"/>
     <joint name="head_camera" type="fixed">

File: aml_sawyer_sim/sawyer_sim_description/urdf/sawyer.xacro (robot description, xacro)
@@ -20,8 +20,22 @@
   <!-- ros_control plugin -->
   <gazebo>
-    <plugin name="gazebo_ros_control" filename="libgazebo_ros_control.so">
+    <plugin name="sawyer_limb_control" filename="libgazebo_ros_control.so">
     <robotNamespace>/robot</robotNamespace>
-    <robotSimType>gazebo_ros_control/DefaultRobotHWSim</robotSimType>
+    <!-- <robotSimType>gazebo_ros_control/DefaultRobotHWSim</robotSimType> -->
     </plugin>
   </gazebo>
+  <gazebo>
+    <plugin name="sawyer_effector_control" filename="libgazebo_ros_control.so">
+    <robotNamespace>/io</robotNamespace>
+    </plugin>
+  </gazebo>
+  <gazebo reference="head_display">
+    <visual>
+      <plugin name="screen_video_controller" filename="libgazebo_ros_video.so">
+        <height>600</height>
+        <width>1024</width>
+        <topicName>/robot/head_display</topicName>
+      </plugin>
+    </visual>
+  </gazebo>
 </robot>

Commit message: updated gazebo control plugin

File: aml_sawyer_sim/sawyer_sim_description/urdf/sawyer.transmission.xacro (robot description, xacro)
@@ -82,24 +82,4 @@
       </actuator>
     </transmission>
-    <transmission name="r_gripper_l_finger_trans">
-      <type>transmission_interface/SimpleTransmission</type>
-      <joint name="r_gripper_l_finger_joint">
-        <hardwareInterface>EffortJointInterface</hardwareInterface>
-      </joint>
-      <actuator name="r_gripper_l_finger_motor">
-        <mechanicalReduction>1</mechanicalReduction>
-        <hardwareInterface>EffortJointInterface</hardwareInterface>
-      </actuator>
-    </transmission>
-    <transmission name="r_gripper_r_finger_trans">
-      <type>transmission_interface/SimpleTransmission</type>
-      <joint name="r_gripper_r_finger_joint">
-        <hardwareInterface>EffortJointInterface</hardwareInterface>
-      </joint>
-      <actuator name="r_gripper_r_finger_motor">
-        <mechanicalReduction>1</mechanicalReduction>
-        <hardwareInterface>EffortJointInterface</hardwareInterface>
-      </actuator>
-    </transmission>
   </xacro:macro>
 </robot>

File: aml_sawyer_sim/sawyer_sim_description/urdf/sawyer.xacro (robot description, xacro)
@@ -20,12 +20,11 @@
   <!-- ros_control plugin -->
   <gazebo>
-    <plugin name="sawyer_limb_control" filename="libgazebo_ros_control.so">
-    <robotNamespace>/robot</robotNamespace>
-    <!-- <robotSimType>gazebo_ros_control/DefaultRobotHWSim</robotSimType> -->
+    <plugin name="sawyer_arm_control" filename="libsawyer_gazebo_ros_control.so">
+      <robotNamespace>/robot</robotNamespace>
     </plugin>
   </gazebo>
   <gazebo>
-    <plugin name="sawyer_effector_control" filename="libgazebo_ros_control.so">
-    <robotNamespace>/io</robotNamespace>
+    <plugin name="sawyer_effector_control" filename="libintera_gripper_gazebo_ros_control.so">
+      <robotNamespace>/io</robotNamespace>
     </plugin>
   </gazebo>
@@ -39,3 +38,31 @@
     </visual>
   </gazebo>
+   <!-- Gazebo-Specific Link Properties -->
+  <gazebo reference="torso">
+    <selfCollide>true</selfCollide>
+  </gazebo>
+  <gazebo reference="head_pan">
+    <implicitSpringDamper>1</implicitSpringDamper>
+  </gazebo>
+  <gazebo reference="right_0">
+    <implicitSpringDamper>1</implicitSpringDamper>
+  </gazebo>
+  <gazebo reference="right_1">
+    <implicitSpringDamper>1</implicitSpringDamper>
+  </gazebo>
+  <gazebo reference="right_2">
+    <implicitSpringDamper>1</implicitSpringDamper>
+  </gazebo>
+  <gazebo reference="right_3">
+    <implicitSpringDamper>1</implicitSpringDamper>
+  </gazebo>
+  <gazebo reference="right_4">
+    <implicitSpringDamper>1</implicitSpringDamper>
+  </gazebo>
+  <gazebo reference="right_5">
+    <implicitSpringDamper>1</implicitSpringDamper>
+  </gazebo>
+  <gazebo reference="right_6">
+    <implicitSpringDamper>1</implicitSpringDamper>
+  </gazebo>
 </robot>
