Commit message: sawyer's ik_pick_and_place works like as baxter's one

File: aml_sawyer_sim/sawyer_sim_description/urdf/sawyer.xacro (robot description, xacro)
@@ -4,5 +4,4 @@
   <xacro:include filename="$(find sawyer_sim_description)/urdf/sawyer_stand.urdf.xacro" />
   <xacro:include filename="$(find intera_tools_description)/urdf/electric_gripper/rethink_electric_gripper.xacro" />
-  <!--<xacro:include filename="$(find intera_tools_description)/urdf/pneumatic_gripper/rethink_pneumatic_gripper.xacro" />-->
   <xacro:sawyer_robot real_mass="true"/>
   <xacro:sawyer_stand />
@@ -17,5 +16,4 @@
                                   r_finger_grasp="inner"
                                   use_connector_plate="True"/>
-  <!--<xacro:rethink_pneumatic_gripper side="right"/>-->
   <!-- ros_control plugin -->
   <gazebo>
@@ -66,3 +64,12 @@
     <implicitSpringDamper>1</implicitSpringDamper>
   </gazebo>
+  <!-- ode param -->
+  <gazebo reference="r_gripper_f_fingr_tip">
+    <mu1>1000</mu1>
+    <mu2>1000</mu2>
+  </gazebo>
+  <gazebo reference="r_gripper_l_fingr_tip">
+    <mu1>1000</mu1>
+    <mu2>1000</mu2>
+  </gazebo>
 </robot>

File: aml_sawyer_sim/sawyer_sim_description/urdf/sawyer_stand.urdf.xacro (robot description, xacro)
@@ -39,4 +39,7 @@
       </inertial>
     </link>
+    <gazebo reference="pedestal">
+      <material>Gazebo/FlatBlack</material>
+    </gazebo>
     <link name="controller_box">
       <collision>

File: aml_sawyer_sim/sawyer_sim_examples/models/block/model.urdf (robot description, URDF)
Before this commit: robot block, 1 links, 0 joints
Links:
- link block: geometry collision box size=0.05 0.03 0.05; visual box size=0.05 0.03 0.05
