Commit message: pih world demo with motor input for 3dof arm

File: aml_playground/src/aml_playground/peg_in_hole/pih_worlds/bullet/models/pih_setup/3_link_planar_arm.urdf (robot description, URDF)
Before this commit: robot test_robot, 4 links, 3 joints
Links:
- link link1: geometry collision cylinder length=0.2 radius=0.05; visual cylinder length=0.2 radius=0.05
Joints:
- joint joint1: axis 1 0 0 -> 0 0 1
- joint joint2: origin xyz=0 0 0.5 rpy=0 0 0 -> xyz=0 0 0.2 rpy=0 0 0

File: aml_playground/src/aml_playground/peg_in_hole/pih_worlds/bullet/models/pih_setup/square_hole.urdf (robot description, URDF)
Before this commit: robot square_hole, 6 links, 5 joints
Links:
- added link groove_base, mass 10; collision box size=2.7 0.7 0.3; visual box size=2.7 0.7 0.3
- added link groove_side1, mass 10; collision box size=2.7 0.3 0.6; visual box size=2.7 0.3 0.6
- added link groove_side2, mass 10; collision box size=2.7 0.3 0.6; visual box size=2.7 0.3 0.6
Joints:
- added joint table_to_groove1: type fixed, parent table, child groove_side1, origin xyz=1.85 0.5 0
- added joint table_to_groove2: type fixed, parent table, child groove_side2, origin xyz=1.85 -0.5 0
- added joint table_to_groove_base: type fixed, parent table, child groove_base, origin xyz=1.85 0 0

Commit message: trial file to check traj following

File: aml_playground/src/aml_playground/peg_in_hole/pih_worlds/bullet/models/pih_setup/3_link_planar_arm.urdf (robot description, URDF)
Before this commit: robot test_robot, 4 links, 3 joints
Links:
- added link eePoint, mass 0.001; collision sphere radius=0.05; visual sphere radius=0.05
Joints:
- added joint joint4: type fixed, parent link3, child eePoint, origin xyz=0. 0. 0.5

Commit message: cleaned some of the codes

File: aml_playground/src/aml_playground/peg_in_hole/pih_worlds/bullet/models/pih_setup/3_link_planar_arm.urdf (robot description, URDF)
Before this commit: robot test_robot, 5 links, 4 joints
Links:
- link link1: geometry collision capsule length=0.2 radius=0.05; visual capsule length=0.2 radius=0.05
- link link2: geometry collision capsule length=0.5 radius=0.05; visual capsule length=0.5 radius=0.05
- link link3: geometry collision capsule length=0.5 radius=0.05; visual capsule length=0.5 radius=0.05
