Commit message: sawyer with pisa hand descriptions and cleaning of bullet robot

File: aml_rl/aml_rl_envs/src/aml_rl_envs/models/sawyer/sawyer_with_pisa_hand.urdf.xacro (robot description, xacro)
@@ -425,86 +425,4 @@
     <axis xyz="0 0 0"/>
   </joint>
-  <!--
-  <transmission name="right_j0_trans">
-    <type>transmission_interface/SimpleTransmission</type>
-    <joint name="right_j0">
-      <hardwareInterface>EffortJointInterface</hardwareInterface>
-    </joint>
-    <actuator name="right_j0_motor">
-      <mechanicalReduction>1</mechanicalReduction>
-      <hardwareInterface>EffortJointInterface</hardwareInterface>
-    </actuator>
-  </transmission>
-  <transmission name="right_j1_trans">
-    <type>transmission_interface/SimpleTransmission</type>
-    <joint name="right_j1">
-      <hardwareInterface>EffortJointInterface</hardwareInterface>
-    </joint>
-    <actuator name="right_j1_motor">
-      <mechanicalReduction>1</mechanicalReduction>
-      <hardwareInterface>EffortJointInterface</hardwareInterface>
-    </actuator>
-  </transmission>
-  <transmission name="right_j2_trans">
-    <type>transmission_interface/SimpleTransmission</type>
-    <joint name="right_j2">
-      <hardwareInterface>EffortJointInterface</hardwareInterface>
-    </joint>
-    <actuator name="right_j2_motor">
-      <mechanicalReduction>1</mechanicalReduction>
-      <hardwareInterface>EffortJointInterface</hardwareInterface>
-    </actuator>
-  </transmission>
-  <transmission name="right_j3_trans">
-    <type>transmission_interface/SimpleTransmission</type>
-    <joint name="right_j3">
-      <hardwareInterface>EffortJointInterface</hardwareInterface>
-    </joint>
-    <actuator name="right_j3_motor">
-      <mechanicalReduction>1</mechanicalReduction>
-      <hardwareInterface>EffortJointInterface</hardwareInterface>
-    </actuator>
-  </transmission>
-  <transmission name="right_j4_trans">
-    <type>transmission_interface/SimpleTransmission</type>
-    <joint name="right_j4">
-      <hardwareInterface>EffortJointInterface</hardwareInterface>
-    </joint>
-    <actuator name="right_j4_motor">
-      <mechanicalReduction>1</mechanicalReduction>
-      <hardwareInterface>EffortJointInterface</hardwareInterface>
-    </actuator>
-  </transmission>
-  <transmission name="right_j5_trans">
-    <type>transmission_interface/SimpleTransmission</type>
-    <joint name="right_j5">
-      <hardwareInterface>EffortJointInterface</hardwareInterface>
-    </joint>
-    <actuator name="right_j5_motor">
-      <mechanicalReduction>1</mechanicalReduction>
-      <hardwareInterface>EffortJointInterface</hardwareInterface>
-    </actuator>
-  </transmission>
-  <transmission name="right_j6_trans">
-    <type>transmission_interface/SimpleTransmission</type>
-    <joint name="right_j6">
-      <hardwareInterface>EffortJointInterface</hardwareInterface>
-    </joint>
-    <actuator name="right_j6_motor">
-      <mechanicalReduction>1</mechanicalReduction>
-      <hardwareInterface>EffortJointInterface</hardwareInterface>
-    </actuator>
-  </transmission>
-  <transmission name="head_pan_trans">
-    <type>transmission_interface/SimpleTransmission</type>
-    <joint name="head_pan">
-      <hardwareInterface>EffortJointInterface</hardwareInterface>
-    </joint>
-    <actuator name="head_pan_motor">
-      <mechanicalReduction>1</mechanicalReduction>
-      <hardwareInterface>EffortJointInterface</hardwareInterface>
-    </actuator>
-  </transmission>
--->
   <link name="base"/>
   <link name="torso">
@@ -544,9 +462,4 @@
     </inertial>
   </link>
-  <!--
-  <gazebo reference="pedestal">
-    <material>Gazebo/FlatBlack</material>
-  </gazebo>
--->
   <link name="controller_box">
     <collision>
@@ -590,258 +503,8 @@
     <child link="right_arm_base_link"/>
   </joint>
-  <!-- Base of end effector -->
-  <link name="right_gripper_base">
-    <inertial>
-      <origin rpy="0 0 0" xyz="0 0 0"/>
-      <mass value="0.0001"/>
-      <inertia ixx="0" ixy="0" ixz="0" iyy="0" iyz="0" izz="0.0"/>
-    </inertial>
-  </link>
-  <!-- Electric Gripper Base Link -->
-  <link name="right_electric_gripper_base">
-    <visual>
-      <origin rpy="0 0 0" xyz="0 0 0"/>
-      <geometry>
-        <mesh filename="meshes/electric_gripper/electric_gripper_base.DAE"/>
-      </geometry>
-    </visual>
-    <collision>
-      <origin rpy="-1.57079632679 3.14159265359 0" xyz="0.004 0.0 0.025"/>
-      <geometry>
-        <cylinder length="0.1" radius="0.029"/>
-      </geometry>
-      <material name="darkred">
-        <color rgba=".5 .1 .1 1"/>
-      </material>
-    </collision>
-    <inertial>
-      <origin rpy="-1.57079632679 3.14159265359 0" xyz="0.0 0.0 0.0"/>
-      <!-- gripper_base mass -->
-      <mass value="0.3"/>
-      <inertia ixx="2e-08" ixy="0" ixz="0" iyy="3e-08" iyz="0" izz="2e-08"/>
-    </inertial>
-  </link>
-  <!-- Connector Plate Joint -->
-  <joint name="right_connector_plate_joint" type="fixed">
-    <origin rpy="0 0 0" xyz="0 0 0"/>
-    <parent link="right_gripper_base"/>
-    <child link="right_connector_plate_base"/>
-  </joint>
-  <link name="right_connector_plate_base">
-    <inertial>
-      <origin rpy="0 0 0" xyz="-0.00032768 -2.5612E-05 0.0062193"/>
-      <mass value="0.1609"/>
-      <inertia ixx="6.9922E-05" ixy="6.1026E-08" ixz="-1.7042E-06" iyy="6.8188E-05" iyz="-1.6118E-08" izz="0.00012392"/>
-    </inertial>
-    <visual>
-      <origin rpy="0 0 0" xyz="0 0 0"/>
-      <geometry>
-        <mesh filename="meshes/connector_plate/connector_plate.STL"/>
-      </geometry>
-      <material name="black">
-        <color rgba="0.05 0.05 0.05 1"/>
-      </material>
-    </visual>
-    <collision>
-      <origin rpy="0 0 0" xyz="0 0 0.0135"/>
-      <geometry>
-        <cylinder length="0.0302" radius="0.04"/>
-      </geometry>
-      <material name="darkred">
-        <color rgba=".5 .1 .1 1"/>
-      </material>
-    </collision>
-  </link>
-  <link name="right_connector_plate_mount"/>
-  <joint name="right_connector_plate_base_joint" type="fixed">
-    <origin rpy="0 0 0" xyz="0 0 0.0151"/>
-    <parent link="right_connector_plate_base"/>
-    <child link="right_connector_plate_mount"/>
-  </joint>
-  <!-- Electric Gripper Base joint -->
-  <joint name="right_electric_gripper_base_jnt" type="fixed">
-    <origin rpy="0 0 0" xyz="0 0 0"/>
-    <parent link="right_connector_plate_mount"/>
-    <child link="right_electric_gripper_base"/>
-  </joint>
-  <link name="r_gripper_l_finger">
-    <visual>
-      <origin rpy="0 0 -3.14159265359" xyz="0 0 0"/>
-      <geometry>
-        <mesh filename="meshes/electric_gripper/fingers/standard_narrow.DAE"/>
-      </geometry>
-    </visual>
-    <collision>
-      <origin rpy="0 0 -3.14159265359" xyz="0 0.01725 0.04"/>
-      <geometry>
-        <box size="0.01 0.0135 0.075"/>
-      </geometry>
-    </collision>
-    <collision>
-      <origin rpy="0 0 -3.14159265359" xyz="-0.005 -0.003 0.0083"/>
-      <geometry>
-        <box size="0.01 0.05 0.017"/>
-      </geometry>
-    </collision>
-    <inertial>
-      <origin rpy="0 0 -3.14159265359" xyz="0 0 0"/>
-      <mass value="0.02"/>
-      <inertia ixx="0.01" ixy="0" ixz="0" iyy="0.01" iyz="0" izz="0.01"/>
-    </inertial>
-  </link>
-  <!--
-  <gazebo reference="r_gripper_l_finger">
-    <mu1>1000</mu1>
-    <mu2>1000</mu2>
-    <fdir1>0.0 0.0 1.0</fdir1>
-    <kp>1e5</kp>
-    <kd>1.0</kd>
-  </gazebo>
--->
-  <link name="r_gripper_l_finger_tip">
-    <visual>
-      <origin rpy="0 0 3.14159265359" xyz="0 0 0"/>
-      <geometry>
-        <mesh filename="meshes/electric_gripper/fingers/paddle_tip.DAE"/>
-      </geometry>
-    </visual>
-    <collision>
-      <origin rpy="0 0 3.14159265359" xyz="0 -0.0045 -0.015"/>
-      <geometry>
-        <box size="0.042 0.0065 0.037"/>
-      </geometry>
-    </collision>
-    <inertial>
-      <origin rpy="0 0 3.14159265359" xyz="0 0 0"/>
-      <mass value="0.01"/>
-      <inertia ixx="0.01" ixy="0" ixz="0" iyy="0.01" iyz="0" izz="0.01"/>
-    </inertial>
-  </link>
-  <joint name="r_gripper_l_finger_tip_joint" type="fixed">
-    <origin rpy="0 0 0" xyz="0.0 0.01725 0.075"/>
-    <parent link="r_gripper_l_finger"/>
-    <child link="r_gripper_l_finger_tip"/>
-  </joint>
-  <link name="r_gripper_r_finger">
-    <visual>
-      <origin rpy="0 0 -0.0" xyz="0 0 0"/>
-      <geometry>
-        <mesh filename="meshes/electric_gripper/fingers/standard_narrow.DAE"/>
-      </geometry>
-    </visual>
-    <collision>
-      <origin rpy="0 0 -0.0" xyz="0 -0.01725 0.04"/>
-      <geometry>
-        <box size="0.01 0.0135 0.075"/>
-      </geometry>
-    </collision>
-    <collision>
-      <origin rpy="0 0 -0.0" xyz="0.005 0.003 0.0083"/>
-      <geometry>
-        <box size="0.01 0.05 0.017"/>
-      </geometry>
-    </collision>
-    <inertial>
-      <origin rpy="0 0 -0.0" xyz="0 0 0"/>
-      <mass value="0.02"/>
-      <inertia ixx="0.01" ixy="0" ixz="0" iyy="0.01" iyz="0" izz="0.01"/>
-    </inertial>
-  </link>
-  <!--
-  <gazebo reference="r_gripper_r_finger">
-    <mu1>1000</mu1>
-    <mu2>1000</mu2>
-    <fdir1>0.0 0.0 1.0</fdir1>
-    <kp>1e5</kp>
-    <kd>1.0</kd>
-  </gazebo>
--->
-  <link name="r_gripper_r_finger_tip">
-    <visual>
-      <origin rpy="0 0 0.0" xyz="0 0 0"/>
-      <geometry>
-        <mesh filename="meshes/electric_gripper/fingers/paddle_tip.DAE"/>
-      </geometry>
-    </visual>
-    <collision>
-      <origin rpy="0 0 0.0" xyz="0 0.0045 -0.015"/>
-      <geometry>
-        <box size="0.042 0.0065 0.037"/>
-      </geometry>
-    </collision>
-    <inertial>
-      <origin rpy="0 0 0.0" xyz="0 0 0"/>
-      <mass value="0.01"/>
-      <inertia ixx="0.01" ixy="0" ixz="0" iyy="0.01" iyz="0" izz="0.01"/>
-    </inertial>
-  </link>
-  <joint name="r_gripper_r_finger_tip_joint" type="fixed">
-    <origin rpy="0 0 0" xyz="0.0 -0.01725 0.075"/>
-    <parent link="r_gripper_r_finger"/>
-    <child link="r_gripper_r_finger_tip"/>
-  </joint>
-  <!-- Gripper Base Joint -->
-  <joint name="right_gripper_base" type="fixed">
-    <origin rpy="0 0 0" xyz="0 0 0"/>
-    <parent link="right_hand"/>
-    <child link="right_gripper_base"/>
-  </joint>
-  <joint name="right_endpoint" type="fixed">
-    <origin rpy="0 0 0" xyz="0 0 0.13562"/>
-    <parent link="right_gripper_base"/>
-    <child link="right_gripper"/>
-  </joint>
-  <!-- Electric Gripper Tip link -->
-  <link name="right_gripper">
-    <inertial>
-      <origin rpy="0 0 0" xyz="0 0 0"/>
-      <mass value="0.0001"/>
-      <inertia ixx="0" ixy="0" ixz="0" iyy="0" iyz="0" izz="0.0"/>
-    </inertial>
-  </link>
-  <joint name="r_gripper_l_finger_joint" type="prismatic">
-    <origin rpy="0 0 0" xyz="0.003 -0.0015 0.04552"/>
-    <axis xyz="0 1 0"/>
-    <parent link="right_electric_gripper_base"/>
-    <child link="r_gripper_l_finger"/>
-    <limit effort="20.0" lower="0.0" upper="0.020833" velocity="5.0"/>
-    <dynamics damping="0.7" friction="0.0"/>
-  </joint>
-  <joint name="r_gripper_r_finger_joint" type="prismatic">
-    <origin rpy="0 0 0" xyz="0.003 0.0015 0.04552"/>
-    <axis xyz="0 1 0"/>
-    <parent link="right_electric_gripper_base"/>
-    <child link="r_gripper_r_finger"/>
-    <limit effort="20.0" lower="-0.020833" upper="0.0" velocity="5.0"/>
-    <mimic joint="r_gripper_l_finger_joint" multiplier="-1.0"/>
-    <dynamics damping="0.7" friction="0.0"/>
-  </joint>
-  <!--
-  <transmission name="gripper_right1">
-    <type>transmission_interface/SimpleTransmission</type>
-    <joint name="r_gripper_r_finger_joint">
-      <hardwareInterface>EffortJointInterface</hardwareInterface>
-    </joint>
-    <actuator name="gripper_r1_motor1">
-      <hardwareInterface>EffortJointInterface</hardwareInterface>
-      <mechanicalReduction>1</mechanicalReduction>
-    </actuator>
-  </transmission>
-  <transmission name="gripper_right2">
-    <type>transmission_interface/SimpleTransmission</type>
-    <joint name="r_gripper_l_finger_joint">
-      <hardwareInterface>EffortJointInterface</hardwareInterface>
-    </joint>
-    <actuator name="gripper_r1_motor2">
-      <hardwareInterface>EffortJointInterface</hardwareInterface>
-      <mechanicalReduction>1</mechanicalReduction>
-    </actuator>
-  </transmission>
-  <gazebo reference="r_gripper_r_finger_joint">
-    <implicitSpringDamper>1</implicitSpringDamper>
-  </gazebo>
-  <gazebo reference="r_gripper_l_finger_joint">
-    <implicitSpringDamper>1</implicitSpringDamper>
-  </gazebo>
--->
+  <xacro:include filename="$(find soft_hand_description)/model/soft_hand.urdf.xacro"/>
+  <xacro:soft_hand name="soft_hand" parent="right_hand"
+                 withAdaptiveTransmission="false" useMimicTag="true" left="false">
+  <origin xyz="0 0 0" rpy="0 0 0"/>
+  </xacro:soft_hand>
 </robot>
