Commit message: collission added to the peg hole of sawyer

File: aml_rl/aml_rl_envs/src/aml_rl_envs/models/sawyer/sawyer2_with_peg.urdf (robot description, URDF)
Before this commit: robot sawyer, 22 links, 21 joints
Links:
- link right_poking_stick: geometry collision mesh filename=meshes/peg_description/poking_stick.STL scale=0.001 0.001 0.001; visual mesh filename=meshes/peg_description/poking_stick.STL scale=0.001 0.001 0.001
- link right_poking_stick_tip: geometry collision box size=0.001 .001 .001; visual box size=0.001 .001 .001

Commit message: corrected urdf for the poking stick

File: aml_rl/aml_rl_envs/src/aml_rl_envs/models/sawyer/sawyer2_with_peg.urdf (robot description, URDF)
Before this commit: robot sawyer, 22 links, 21 joints
Links:
- link right_poking_stick_tip: geometry visual sphere radius=0.01
- link right_soft_hand_adapter: geometry collision mesh filename=meshes/peg_description/pisa_hand_adapter.STL scale=0.001 0.001 0.001; visual mesh filename=meshes/peg_description/pisa_hand_adapter.STL scale=0.001 0.001 0.001
Joints:
- joint right_gripper_soft_hand_adapter: origin xyz=0 0 0.0 rpy=0 0. 0 -> xyz=0.07 -0.04 -0.01 rpy=0 0. 0
- joint right_poking_stick_fixed: origin xyz=0 0 0.0 rpy=0 0. 0 -> xyz=-0.05 0.05 0.03 rpy=0 0. 0
- joint right_poking_stick_tip_fixed: origin xyz=0 0 0. rpy=0 0. 0 -> xyz=0.01 -0.01 0.18 rpy=0 0. 0

Commit message: sawyer peg urdf added

File: aml_rl/aml_rl_envs/src/aml_rl_envs/models/sawyer/sawyer2_with_peg.urdf (robot description, URDF)
Before this commit: robot sawyer, 22 links, 21 joints
Links:
- link right_poking_stick: geometry collision mesh filename=meshes/peg_description/peg_rect1620.STL scale=0.001 0.001 0.001; visual mesh filename=meshes/peg_description/peg_rect1620.STL scale=0.001 0.001 0.001
Joints:
- joint right_poking_stick_fixed: origin xyz=-0.05 0.05 0.03 rpy=0 0. 0 -> xyz=-0.04 0.04 0.03 rpy=0 0. 0
- joint right_poking_stick_tip_fixed: origin xyz=0.01 -0.01 0.18 rpy=0 0. 0 -> xyz=0.0 -0.0 0.177 rpy=0 0. 0

Commit message: urdf file with the peg modified

File: aml_rl/aml_rl_envs/src/aml_rl_envs/models/sawyer/sawyer2_with_peg.urdf (robot description, URDF)
Before this commit: robot sawyer, 22 links, 21 joints
Joints:
- joint head_pan: limit lower=-5.1477 upper=0.9559 effort=8 velocity=1.8 -> (none); type revolute -> fixed
