Commit message: starting up project

File: aml_rl/aml_rl_envs/src/aml_rl_envs/models/sawyer/sawyer.urdf (robot description, URDF)
Before this commit: robot sawyer, 24 links, 23 joints
Joints:
- joint head_pan: type revolute -> fixed

File: aml_rl/aml_rl_envs/src/aml_rl_envs/models/sawyer/sawyer2.urdf (robot description, URDF)
Before this commit: robot sawyer, 19 links, 18 joints
Joints:
- joint head_pan: type revolute -> fixed
