Commit message: modified cylinder urdf to have continous joint

File: aml_rl/aml_rl_envs/src/aml_rl_envs/models/cylinder.urdf (robot description, URDF)
Before this commit: robot robot, 3 links, 2 joints
Links:
- link capsuleobject: geometry collision cylinder length=0.65 radius=0.30; visual cylinder length=0.65 radius=0.30
Joints:
- joint joint1: type fixed -> continuous
