Commit message: increased the diameter of the finger base

File: aml_rl/aml_rl_envs/src/aml_rl_envs/models/hand/four_finger_hand.urdf (robot description, URDF)
Before this commit: robot robot, 17 links, 16 joints
Links:
- link base_link: geometry collision cylinder length=0.05 radius=0.8; visual cylinder length=0.05 radius=0.8
- link f1_eePoint: geometry collision capsule length=0.08 radius=0.05; visual capsule length=0.08 radius=0.05
- link f2_eePoint: geometry collision capsule length=0.08 radius=0.05; visual capsule length=0.08 radius=0.05
- link f3_eePoint: geometry collision capsule length=0.08 radius=0.05; visual capsule length=0.08 radius=0.05
- link f4_eePoint: geometry collision capsule length=0.08 radius=0.05; visual capsule length=0.08 radius=0.05
Joints:
- joint f1_joint1: origin xyz=0.45 0 0. rpy=0 0 0 -> xyz=0.75 0 0. rpy=0 0 0
- joint f1_joint2: limit lower=-1.21619 upper=1.21619 effort=300 velocity=1.0 -> lower=-1.576 upper=1.576 effort=300 velocity=1.0; origin xyz=0 0 0.2 rpy=0 0 0 -> xyz=0. 0 0.2 rpy=0 0 0
- joint f1_joint3: limit lower=-1.97019 upper=2.200 effort=300 velocity=1.0 -> lower=-2.97019 upper=2.900 effort=300 velocity=1.0; origin xyz=0 0 0.5 rpy=0 0 0 -> xyz=0. 0 0.5 rpy=0 0 0
- joint f2_joint1: origin xyz=0 0.45 0 rpy=0 0 1.5707963267948966 -> xyz=0 0.75 0 rpy=0 0 1.5707963267948966
- joint f2_joint3: limit lower=-1.97019 upper=2.200 effort=300 velocity=1.0 -> lower=-2.97019 upper=2.900 effort=300 velocity=1.0
- joint f3_joint1: origin xyz=-0.45 0 0 rpy=0 0 3.14159 -> xyz=-0.75 0 0 rpy=0 0 3.14159
- joint f3_joint3: limit lower=-1.97019 upper=2.200 effort=300 velocity=1.0 -> lower=-2.97019 upper=2.900 effort=300 velocity=1.0
- joint f4_joint1: origin xyz=0 -0.45 0 rpy=0 0 -1.5707963267948966 -> xyz=0 -0.75 0 rpy=0 0 -1.5707963267948966
- joint f4_joint3: limit lower=-1.97019 upper=2.200 effort=300 velocity=1.0 -> lower=-2.97019 upper=2.900 effort=300 velocity=1.0
