Commit message: sawyer env modified

File: aml_rl/aml_rl_envs/src/aml_rl_envs/models/peg_hole/square_hole_vertical_18x22.urdf (robot description, URDF)
Before this commit: robot square_hole, 5 links, 4 joints
Links:
- link side3: geometry collision box size=0.18 0.66 0.8; visual box size=0.18 0.66 0.8
