Commit message: collision mesh fix

File: aml_grasp/src/aml_grasp/models/mug.urdf (robot description, URDF)
Before this commit: robot mug.urdf, 1 links, 0 joints
Links:
- link mug_link: geometry collision mesh filename=9_Mug/9_a_Ceramic_mugs/conic_with_open_handle.stl scale=1 1 1; visual mesh filename=9_Mug/9_a_Ceramic_mugs/conic_with_open_handle.stl scale=1 1 1
