Commit message: kinmatics updates, urdf with no mass for sawyer, updating pisaiit interface, and many fixes

File: aml_grasp/src/aml_grasp/models/pisa_iit_hand/pisa_hand_left.urdf (robot description, URDF)
Before this commit: robot soft_hand, 40 links, 39 joints
Links:
- removed link hand
- added link right_hand

File: aml_grasp/src/aml_grasp/models/pisa_iit_hand/pisa_hand_right.urdf (robot description, URDF)
Before this commit: robot soft_hand, 40 links, 39 joints
Links:
- removed link hand
- added link right_hand
Joints:
- joint hand_soft_hand_kuka_coupler_joint: parent hand -> right_hand

File: aml_grasp/src/aml_grasp/models/sawyer/sawyer2_with_pisa_hand.urdf.xacro (robot description, xacro)
@@ -437,5 +437,5 @@
   <xacro:include filename="$(find soft_hand_description)/model/soft_hand.urdf.xacro"/>
   <xacro:soft_hand name="soft_hand" parent="right_hand"
-                 withAdaptiveTransmission="false" useMimicTag="true" left="false">
+                 withAdaptiveTransmission="true" useMimicTag="true" left="false">
   <origin xyz="0 0 0" rpy="0 0 0"/>
   </xacro:soft_hand>

File: aml_grasp/src/aml_grasp/models/sawyer/sawyer_with_pisa_hand.urdf.xacro (robot description, xacro)
@@ -505,5 +505,5 @@
   <xacro:include filename="$(find soft_hand_description)/model/soft_hand.urdf.xacro"/>
   <xacro:soft_hand name="soft_hand" parent="right_hand"
-                 withAdaptiveTransmission="false" useMimicTag="true" left="false">
+                 withAdaptiveTransmission="true" useMimicTag="true" left="false">
   <origin xyz="0 0 0" rpy="0 0 0"/>
   </xacro:soft_hand>
