Commit message: fixing robot descriptions

File: aml_grasp/src/aml_grasp/models/pisa_iit_hand/pisa_hand_right_nofake_links.urdf (robot description, URDF)
Before this commit: robot pisa_iit, 40 links, 39 joints
Links:
- removed link soft_hand_index_fake_link1
- removed link soft_hand_index_fake_link2
- removed link soft_hand_index_fake_link3
- removed link soft_hand_little_fake_link1
- removed link soft_hand_little_fake_link2
- removed link soft_hand_little_fake_link3
- removed link soft_hand_middle_fake_link1
- removed link soft_hand_middle_fake_link2
- removed link soft_hand_middle_fake_link3
- removed link soft_hand_ring_fake_link1
- removed link soft_hand_ring_fake_link2
- removed link soft_hand_ring_fake_link3
- removed link soft_hand_thumb_fake_link1
- removed link soft_hand_thumb_fake_link3
Joints:
- removed joint soft_hand_index_inner_joint_mimic
- removed joint soft_hand_index_middle_joint_mimic
- removed joint soft_hand_index_outer_joint_mimic
- removed joint soft_hand_little_inner_joint_mimic
- removed joint soft_hand_little_middle_joint_mimic
- removed joint soft_hand_little_outer_joint_mimic
- removed joint soft_hand_middle_inner_joint_mimic
- removed joint soft_hand_middle_middle_joint_mimic
- removed joint soft_hand_middle_outer_joint_mimic
- removed joint soft_hand_ring_inner_joint_mimic
- removed joint soft_hand_ring_middle_joint_mimic
- removed joint soft_hand_ring_outer_joint_mimic
- removed joint soft_hand_thumb_inner_joint_mimic
- removed joint soft_hand_thumb_outer_joint_mimic
- joint soft_hand_index_inner_joint: child soft_hand_index_fake_link1 -> soft_hand_index_proximal_link
- joint soft_hand_index_middle_joint: child soft_hand_index_fake_link2 -> soft_hand_index_middle_link
- joint soft_hand_index_outer_joint: child soft_hand_index_fake_link3 -> soft_hand_index_distal_link
- joint soft_hand_little_inner_joint: child soft_hand_little_fake_link1 -> soft_hand_little_proximal_link
- joint soft_hand_little_middle_joint: child soft_hand_little_fake_link2 -> soft_hand_little_middle_link
- joint soft_hand_little_outer_joint: child soft_hand_little_fake_link3 -> soft_hand_little_distal_link
- joint soft_hand_middle_inner_joint: child soft_hand_middle_fake_link1 -> soft_hand_middle_proximal_link
- joint soft_hand_middle_middle_joint: child soft_hand_middle_fake_link2 -> soft_hand_middle_middle_link
- joint soft_hand_middle_outer_joint: child soft_hand_middle_fake_link3 -> soft_hand_middle_distal_link
- joint soft_hand_ring_inner_joint: child soft_hand_ring_fake_link1 -> soft_hand_ring_proximal_link
- joint soft_hand_ring_middle_joint: child soft_hand_ring_fake_link2 -> soft_hand_ring_middle_link
- joint soft_hand_ring_outer_joint: child soft_hand_ring_fake_link3 -> soft_hand_ring_distal_link
- joint soft_hand_thumb_inner_joint: child soft_hand_thumb_fake_link1 -> soft_hand_thumb_proximal_link
- joint soft_hand_thumb_outer_joint: child soft_hand_thumb_fake_link3 -> soft_hand_thumb_distal_link

File: aml_grasp/src/aml_grasp/models/sawyer/sawyer2_with_pisa_hand.urdf.xacro (robot description, xacro)
@@ -437,5 +437,5 @@
   <xacro:include filename="$(find soft_hand_description)/model/soft_hand.urdf.xacro"/>
   <xacro:soft_hand name="soft_hand" parent="right_hand"
-                 withAdaptiveTransmission="true" useMimicTag="true" left="false">
+                 withAdaptiveTransmission="false" useMimicTag="false" left="false">
   <origin xyz="0 0 0" rpy="0 0 0"/>
   </xacro:soft_hand>

File: aml_grasp/src/aml_grasp/models/sawyer/sawyer_with_pisa_hand.urdf.xacro (robot description, xacro)
@@ -505,5 +505,5 @@
   <xacro:include filename="$(find soft_hand_description)/model/soft_hand.urdf.xacro"/>
   <xacro:soft_hand name="soft_hand" parent="right_hand"
-                 withAdaptiveTransmission="true" useMimicTag="true" left="false">
+                 withAdaptiveTransmission="false" useMimicTag="false" left="false">
   <origin xyz="0 0 0" rpy="0 0 0"/>
   </xacro:soft_hand>
