Commit message: implementing full robot and updating descriptions

File: aml_grasp/src/aml_grasp/models/pisa_iit_hand/pisa_hand_right_nomass.urdf (robot description, URDF)
Before this commit: robot soft_hand, 39 links, 39 joints
Joints:
- joint hand_soft_hand_kuka_coupler_joint: origin xyz=0.0 0.0 0.0 rpy=0 0 0 -> xyz=0.007 0.0 0.0035 rpy=0 0 -1.570796327
